Commit message: change ackermann calculations to invert based on the new gpio node

File: src/vehicle_bringup/urdf/jetson-car.urdf (robot description, URDF)
Before this commit: robot jetson-car, 6 links, 5 joints
Links:
- link base_link: mass None -> 0.01; geometry 
- link chassis: mass None -> 1.0; geometry collision box size=0.20 0.10 0.05; visual box size=0.20 0.10 0.05
- link front_left_wheel: mass None -> 0.1; geometry collision cylinder length=0.02 radius=0.034; visual cylinder length=0.02 radius=0.034
- link front_right_wheel: mass None -> 0.1; geometry collision cylinder length=0.02 radius=0.034; visual cylinder length=0.02 radius=0.034
- link rear_left_wheel: mass None -> 0.1; geometry collision cylinder length=0.02 radius=0.034; visual cylinder length=0.02 radius=0.034
- link rear_right_wheel: mass None -> 0.1; geometry collision cylinder length=0.02 radius=0.034; visual cylinder length=0.02 radius=0.034

Commit message: fixed ai lane detection, added launch arguements, added gazebo world, install script for gpu activation on the jetson

File: src/vehicle_bringup/urdf/jetson-car.urdf (robot description, URDF)
Before this commit: robot jetson-car, 6 links, 5 joints
Links:
- added link camera_link; visual box size=0.02 0.04 0.02
- added link fl_steering_hinge, mass 0.05
- added link fr_steering_hinge, mass 0.05
Joints:
- added joint camera_joint: type fixed, parent base_link, child camera_link, origin xyz=0.174 0 0.04 rpy=0 0 0
- added joint fl_steering_joint: type revolute, parent base_link, child fl_steering_hinge, origin xyz=0.148 0.0665 0.034 rpy=0 0 0, axis 0 0 1, limit lower=-0.52 upper=0.52 effort=10.0 velocity=5.0
- added joint fr_steering_joint: type revolute, parent base_link, child fr_steering_hinge, origin xyz=0.148 -0.0665 0.034 rpy=0 0 0, axis 0 0 1, limit lower=-0.52 upper=0.52 effort=10.0 velocity=5.0
- joint fl_wheel_joint: origin xyz=0.148 0.0665 0.034 rpy=0 0 0 -> xyz=0 0 0 rpy=0 0 0; parent base_link -> fl_steering_hinge
- joint fr_wheel_joint: origin xyz=0.148 -0.0665 0.034 rpy=0 0 0 -> xyz=0 0 0 rpy=0 0 0; parent base_link -> fr_steering_hinge

Commit message: all the sim work i did over march, im sorry ill lock in with commits

File: src/vehicle_bringup/urdf/jetson-car.urdf (robot description, URDF)
Before this commit: robot jetson-car, 9 links, 8 joints
Links:
- link chassis: geometry collision box size=0.2413 0.10 0.05; visual box size=0.2413 0.10 0.05
Joints:
- joint camera_joint: origin xyz=0.174 0 0.04 rpy=0 0 0 -> xyz=0.174 0 0.0587 rpy=0 0 0
- joint fl_steering_joint: limit lower=-0.52 upper=0.52 effort=10.0 velocity=5.0 -> lower=-0.785 upper=0.785 effort=10.0 velocity=5.0
- joint fr_steering_joint: limit lower=-0.52 upper=0.52 effort=10.0 velocity=5.0 -> lower=-0.785 upper=0.785 effort=10.0 velocity=5.0
