Commit message: hardware controller spawning and joint spawning worked, now working on bridging actual hardware to controller

File: src/vehicle_bringup/urdf/jetson_car_core.xacro (robot description, xacro)
@@ -4,8 +4,4 @@
   <material name="black"><color rgba="0 0 0 1"/></material>
   <link name="base_link">
-    <inertial>
-      <mass value="0.01"/>
-      <inertia ixx="0.0001" ixy="0" ixz="0" iyy="0.0001" iyz="0" izz="0.0001"/>
-    </inertial>
   </link>
   <link name="chassis">
