Commit message: redid all launch files, fixed tf issues, added headless gazebo compatibility (show_sim=false), added 2 rviz config files

File: src/vehicle_bringup/urdf/jetson_car.ros2_control.xacro (robot description, xacro)
@@ -5,5 +5,5 @@
       <hardware>
         <xacro:if value="${use_sim}">
-          <plugin>ign_ros2_control/IgnitionSystem</plugin>
+          <plugin>gz_ros2_control/GazeboSimSystem</plugin>
         </xacro:if>
         <xacro:unless value="${use_sim}">
@@ -32,4 +32,12 @@
         <state_interface name="position"/>
       </joint>
+      <joint name="fl_wheel_joint">
+        <state_interface name="position"/>
+        <state_interface name="velocity"/>
+      </joint>
+      <joint name="fr_wheel_joint">
+        <state_interface name="position"/>
+        <state_interface name="velocity"/>
+      </joint>
     </ros2_control>
   </xacro:macro>

Commit message: updated all launch files from old rework branch code, during headless sim, gz needs fluid front wheels but hardware doesnt so added param handling in both urdfs

File: src/vehicle_bringup/urdf/jetson_car.ros2_control.xacro (robot description, xacro)
@@ -32,12 +32,14 @@
         <state_interface name="position"/>
       </joint>
-      <joint name="fl_wheel_joint">
-        <state_interface name="position"/>
-        <state_interface name="velocity"/>
-      </joint>
-      <joint name="fr_wheel_joint">
-        <state_interface name="position"/>
-        <state_interface name="velocity"/>
-      </joint>
+      <xacro:if value="${use_sim}">
+        <joint name="fl_wheel_joint">
+          <state_interface name="position"/>
+          <state_interface name="velocity"/>
+        </joint>
+        <joint name="fr_wheel_joint">
+          <state_interface name="position"/>
+          <state_interface name="velocity"/>
+        </joint>
+      </xacro:if>
     </ros2_control>
   </xacro:macro>

File: src/vehicle_bringup/urdf/jetson_car.urdf.xacro (robot description, xacro)
@@ -7,7 +7,7 @@
   <xacro:if value="$(arg use_sim)">
     <gazebo>
-    <plugin filename="libign_ros2_control-system.so" name="ign_ros2_control::IgnitionROS2ControlPlugin">
-      <parameters>$(find vehicle_hardware)/config/controllers.yaml</parameters>
-    </plugin>
+      <plugin filename="libgz_ros2_control-system.so" name="gz_ros2_control::GazeboSimROS2ControlPlugin">
+        <parameters>$(find vehicle_hardware)/config/controllers.yaml</parameters>
+      </plugin>
       <plugin filename="libignition-gazebo-odometry-publisher-system.so" name="ignition::gazebo::systems::OdometryPublisher">
         <odom_frame>odom</odom_frame>
